File: hardware/ESP-07_tryout/ESP-07_tryout.sch (KiCad schematic (older format))
At the start: 0 parts

Commit message: update,
Parts:
- added J?: Conn_01x04_Female, symbol Connector:Conn_01x04_Female
- added R? (x2): R103,0603, Resistor_SMD:R_0603_1608Metric_Pad1.05x0.95mm_HandSolder, symbol taobao-r:R103,0603
- added U?: ESP-07, footprint-lib:ESP-07, symbol taobao-components:ESP-07
Connections:
- new net: R?.1, U?.1 (RESET)
- new net: J?.3 (Pin_3), U?.15 (RX0/GPIO13)
- new net: J?.2 (Pin_2), U?.16 (TX0/GPIO1)
- new net: R?.1, U?.3 (CH_PD)
- new net +3V3: J?.4 (Pin_4), R?.2, R?.2, U?.8 (VCC)
- new net GND: J?.1 (Pin_1), U?.10 (GPIO15/SS), U?.9 (GND)
